File: RC-CarPCB/_autosave-RC-CarPCB.kicad_pcb (KiCad board)
At the start: 2 copper layers, 90 x 128 mm, 14 parts, among them SW1 SW_SPST, SW2 SW_SPST, SW3 SW_SPST, SW4 SW_SPST, U1 NRF24L01_Breakout

Commit message: stuff
Connections:
- U1 pad 6: Net-(A1-D12) -> Net-(A1-D11)
- U1 pad 7: Net-(A1-D11) -> Net-(A1-D12)
Routing:
- net Net-(A1-D12): track 49.3 -> 34.4 mm, vias 1 -> 2
- net Net-(A1-D11): track 37.0 -> 51.8 mm, vias 2 -> 1
